Commit message: Removed sd vel_switch (redundent) and added lidar to main urdf (lidar shows in rviz by default)

File: src/sdr_frame/config/hk1500.urdf (robot description, URDF)
Before this commit: robot hk_1500, 7 links, 6 joints
Links:
- added link hokuyo_link; collision box size=0.05 0.05 0.07; collision box size=0.079 0.05 0.006
- added link laser_frame
Joints:
- added joint hokuyo_joint: type fixed, parent base_link, child hokuyo_link, origin xyz=0.0775 0 0
- added joint laser_joint: type fixed, parent hokuyo_link, child laser_frame, origin xyz=0 0 0.064

Commit message: updated urdf

File: src/sdr_frame/config/hk1500.urdf (robot description, URDF)
Before this commit: robot hk_1500, 9 links, 8 joints
Links:
- link base_link: mass None -> 83.31; geometry collision box size=0.914 0.53975 0.312; visual box size=0.914 0.53975 0.312
- link fl_wheel_link: mass None -> 9; geometry collision cylinder length=0.108 radius=0.15; visual cylinder length=0.108 radius=0.15
- link fr_wheel_link: mass None -> 9; geometry collision cylinder length=0.108 radius=0.15; visual cylinder length=0.108 radius=0.15
- link ml_wheel_link: mass None -> 9; geometry collision cylinder length=0.108 radius=0.15; visual cylinder length=0.108 radius=0.15
- link mr_wheel_link: mass None -> 9; geometry collision cylinder length=0.108 radius=0.15; visual cylinder length=0.108 radius=0.15
- link rl_wheel_link: mass None -> 9; geometry collision cylinder length=0.108 radius=0.15; visual cylinder length=0.108 radius=0.15
- link rr_wheel_link: mass None -> 9; geometry collision cylinder length=0.108 radius=0.15; visual cylinder length=0.108 radius=0.15
Joints:
- joint ml_wheel_joint: type continuous -> fixed
- joint mr_wheel_joint: type continuous -> fixed
