Commit message: Added Gazebo launch and description package for urdf and future meshes -lidar plugin working

File: src/panther_description/urdf/hk1500.urdf (robot description, URDF)
Before this commit: robot hk_1500, 9 links, 8 joints
Joints:
- joint hokuyo_joint: origin xyz=0.0775 0 0 -> xyz=0.356108 0 0.312
- joint laser_joint: origin xyz=0 0 0.064 -> xyz=0 0 0.376

Commit message: updated urdf with imu

File: src/panther_description/urdf/hk1500.urdf (robot description, URDF)
Before this commit: robot panther, 9 links, 8 joints
Links:
- added link imu_link; collision box size=0.079 0.05 0.006; visual box size=0.079 0.05 0.006
Joints:
- added joint imu_joint: type fixed, parent base_link, child imu_link, origin xyz=0 0 0.449
- joint fl_wheel_joint: origin xyz=0.356108 0.269875 0.0 rpy=-1.5708 0.0 0.0 -> xyz=0.356108 0.269875 0.137 rpy=-1.5708 0.0 0.0
- joint fr_wheel_joint: origin xyz=0.356108 -0.269875 0.0 rpy=1.5708 0.0 0.0 -> xyz=0.356108 -0.269875 0.137 rpy=1.5708 0.0 0.0
- joint hokuyo_joint: origin xyz=0.356108 0 0.312 -> xyz=0.356108 0 0.449
- joint laser_joint: origin xyz=0 0 0.376 -> xyz=0 0 0.513
- joint ml_wheel_joint: origin xyz=0.0 0.269875 0.0 rpy=-1.5708 0.0 0.0 -> xyz=0.0 0.269875 0.137 rpy=-1.5708 0.0 0.0
- joint mr_wheel_joint: origin xyz=0.0 -0.269875 0.0 rpy=1.5708 0.0 0.0 -> xyz=0.0 -0.269875 0.137 rpy=1.5708 0.0 0.0
- joint rl_wheel_joint: origin xyz=-0.356108 0.269875 0.0 rpy=-1.5708 0.0 0.0 -> xyz=-0.356108 0.269875 0.137 rpy=-1.5708 0.0 0.0
- joint rr_wheel_joint: origin xyz=-0.356108 -0.269875 0.0 rpy=1.5708 0.0 0.0 -> xyz=-0.356108 -0.269875 0.137 rpy=1.5708 0.0 0.0

Commit message: Added skid steer plugin (not working)

File: src/panther_description/urdf/hk1500.urdf (robot description, URDF)
Before this commit: robot panther, 10 links, 9 joints
Links:
- added link base_footprint
Joints:
- added joint base_joint: type fixed, parent base_footprint, child base_link, origin xyz=0 0 0.19783 rpy=0 0 0

Commit message: Modified skid steer plugin (still not working) and added cask model to gazebo pkg

File: src/panther_description/urdf/hk1500.urdf (robot description, URDF)
Before this commit: robot panther, 11 links, 10 joints
Joints:
- joint fl_wheel_joint: type fixed -> continuous
- joint fr_wheel_joint: type fixed -> continuous
- joint rl_wheel_joint: type fixed -> continuous
- joint rr_wheel_joint: type fixed -> continuous

Commit message: Update to skidsteer plugin params and link collisions

File: src/panther_description/urdf/hk1500.urdf (robot description, URDF)
Before this commit: robot panther, 11 links, 10 joints
Links:
- link ml_wheel_link: geometry visual cylinder length=0.108 radius=0.15
- link mr_wheel_link: geometry visual cylinder length=0.108 radius=0.15

Commit message: updated urdf joints and other small things

File: src/panther_description/urdf/hk1500.urdf (robot description, URDF)
Before this commit: robot panther, 11 links, 10 joints
Joints:
- joint fl_wheel_joint: axis 0 0 1 -> 0 1 0; origin xyz=0.356108 0.269875 0.137 rpy=-1.5708 0.0 0.0 -> xyz=0.356108 0.323875 0.137
- joint fr_wheel_joint: axis 0 0 1 -> 0 1 0; origin xyz=0.356108 -0.269875 0.137 rpy=1.5708 0.0 0.0 -> xyz=0.356108 -0.323875 0.137
- joint laser_joint: origin xyz=0 0 0.513 -> xyz=0 0 0.04
- joint ml_wheel_joint: axis 0 0 1 -> 0 1 0; origin xyz=0.0 0.269875 0.137 rpy=-1.5708 0.0 0.0 -> xyz=0.0 0.323875 0.137
- joint mr_wheel_joint: axis 0 0 1 -> 0 1 0; origin xyz=0.0 -0.269875 0.137 rpy=1.5708 0.0 0.0 -> xyz=0.0 -0.323875 0.137
- joint rl_wheel_joint: axis 0 0 1 -> 0 1 0; origin xyz=-0.356108 0.269875 0.137 rpy=-1.5708 0.0 0.0 -> xyz=-0.356108 0.323875 0.137
- joint rr_wheel_joint: axis 0 0 1 -> 0 1 0; origin xyz=-0.356108 -0.269875 0.137 rpy=1.5708 0.0 0.0 -> xyz=-0.356108 -0.323875 0.137

Commit message: updated inertia

File: src/panther_description/urdf/hk1500.urdf (robot description, URDF)
Before this commit: robot panther, 11 links, 10 joints
Links:
- link base_link: mass 83.31 -> 55
- link fl_wheel_link: mass 9 -> 6
- link fr_wheel_link: mass 9 -> 6
- link ml_wheel_link: mass 9 -> None
- link mr_wheel_link: mass 9 -> None
- link rl_wheel_link: mass 9 -> 6
- link rr_wheel_link: mass 9 -> 6
Joints:
- joint base_joint: origin xyz=0 0 0.19783 rpy=0 0 0 -> xyz=0 0 0.293 rpy=0 0 0

Commit message: newest updates, there might be an error with the witmotion stuff

File: src/panther_description/urdf/hk1500.urdf (robot description, URDF)
Before this commit: robot panther, 11 links, 10 joints
Links:
- removed link imu_link
- added link imu; collision box size=0.079 0.05 0.006; visual box size=0.079 0.05 0.006
Joints:
- joint base_joint: origin xyz=0 0 0.293 rpy=0 0 0 -> xyz=0 0 0 rpy=0 0 0
- joint fl_wheel_joint: type continuous -> fixed
- joint fr_wheel_joint: type continuous -> fixed
- joint imu_joint: child imu_link -> imu
- joint ml_wheel_joint: type fixed -> continuous
- joint mr_wheel_joint: type fixed -> continuous
- joint rl_wheel_joint: type continuous -> fixed
- joint rr_wheel_joint: type continuous -> fixed

Commit message: updated imu

File: src/panther_description/urdf/hk1500.urdf (robot description, URDF)
Before this commit: robot panther, 11 links, 10 joints
Links:
- removed link imu
- added link imu_link; collision box size=0.079 0.05 0.006; visual box size=0.079 0.05 0.006
Joints:
- joint imu_joint: child imu -> imu_link

Commit message: updated gps

File: src/panther_description/urdf/hk1500.urdf (robot description, URDF)
Before this commit: robot panther, 11 links, 10 joints
Links:
- added link gps; collision box size=0.079 0.05 0.006; visual box size=0.079 0.05 0.006
Joints:
- added joint gps_joint: type fixed, parent base_link, child gps, origin xyz=0 0 0.449
